File: HARDWARE/V2/ant control board v2/sensors.kicad_sch (KiCad schematic)
At the start: 11 parts, among them J8 ADC_AUX, J9 DIGITAL_AUX, U8 LSM6DS3

Commit message: layout 2.0 facv2 done
Parts:
- C10: renamed from C12; footprint Capacitor_SMD:C_0603_1608Metric -> Capacitor_SMD:C_0402_1005Metric; LCSC C282519 -> C1525
- C11: renamed from C13; footprint Capacitor_SMD:C_0603_1608Metric -> Capacitor_SMD:C_0402_1005Metric; LCSC C282519 -> C1525
- C8: renamed from C10; footprint Capacitor_SMD:C_0603_1608Metric -> Capacitor_SMD:C_0402_1005Metric
- C9: renamed from C11; footprint Capacitor_SMD:C_0603_1608Metric -> Capacitor_SMD:C_0402_1005Metric; LCSC C282519 -> C1525
- J10: renamed from J9; footprint _MY_connectors:Pad 02x01 -> _MY_connectors:01x02_TH_pad_renforced_small
- J9: renamed from J8; footprint _MY_connectors:Pad 03x01 -> _MY_connectors:01x03_TH_pad_renforced_small
- R3: renamed from R1; footprint Resistor_SMD:R_0603_1608Metric -> Resistor_SMD:R_0402_1005Metric; LCSC C103199 -> C60490
- R4: renamed from R2; footprint Resistor_SMD:R_0603_1608Metric -> Resistor_SMD:R_0402_1005Metric; LCSC C23186 -> C25867
- R5: renamed from R3; footprint Resistor_SMD:R_0603_1608Metric -> Resistor_SMD:R_0402_1005Metric; LCSC C103199 -> C60490
- R6: renamed from R4; footprint Resistor_SMD:R_0603_1608Metric -> Resistor_SMD:R_0402_1005Metric; LCSC C23186 -> C25905
- renumbered U8 to U5
